Commit message: changes

File: description/robot.urdf.xacro (robot description, xacro)
@@ -1,4 +1,4 @@
    <?xml version="1.0"?>
-<robot xmlns:xacro="http://www.ros.org/wiki/xacro"  name="robot">
+<robot xmlns:xacro="http://www.ros.org/wiki/xacro" name="robot">
     <xacro:include filename="robot_core.xacro" />
 </robot>

File: description/robot_core.xacro (robot description, xacro)
@@ -1,32 +1,26 @@
-<?xml version="1.0"?>
-<robot xmlns:xacro="http://www.ros.org/wiki/xacro">
-    ... all our links and joints will go in here ...
-<material name="white">
-    <color rgba="1 1 1 1"/>
-</material>
-<material name="orange">
-    <color rgba="1 0.3 0.1 1"/>
-</material>
-<material name="blue">
-    <color rgba="0.2 0.2 1 1"/>
-</material>
-<material name="black">
-    <color rgba="0 0 0 1"/>
-</material>
-<link name="base_link">
-</link>
-<joint name="chassis_joint" type="fixed">
-    <parent link="base_link"/>
-    <child link="chassis"/>
-    <origin xyz="-0.1 0 0"/>
-</joint>
-<link name="chassis">
-    <visual>
-        <origin xyz="0.15 0 0.075" rpy="0 0 0"/>
-        <geometry>
-            <box size="0.3 0.3 0.15"/>
-        </geometry>
-        <material name="white"/>
-    </visual>
-</link>
+<robot xmlns:xacro="http://www.ros.org/wiki/xacro" name="robot_core">
+    <material name="orange">
+        <color rgba="1 0.3 0.1 1"/>
+    </material>
+    <material name="blue">
+        <color rgba="0.2 0.2 1 1"/>
+    </material>
+    <material name="black">
+        <color rgba="0 0 0 1"/>
+    </material>
+    <link name="base_link"/>
+    <joint name="chassis_joint" type="fixed">
+        <parent link="base_link"/>
+        <child link="chassis"/>
+        <origin xyz="-0.1 0 0"/>
+    </joint>
+    <link name="chassis">
+        <visual>
+            <origin xyz="0.15 0 0.075" rpy="0 0 0"/>
+            <geometry>
+                <box size="0.3 0.3 0.15"/>
+            </geometry>
+            <material name="white"/>
+        </visual>
+    </link>
 </robot>
